File: 04_sd-card.kicad_sch (KiCad schematic)
At the start: 8 parts, among them J6 Micro_SD_Card_Det2

Commit message: v2: final touch
- add proper ESD diodes for USB
- move the USB fuse right after the connector
- pretty labels for test points
Parts:
- renumbered R16 to R12, R12 to R13, R13 to R14, R14 to R15, R15 to R16
Changed lines of the file:
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@@
 		(on_board yes)
 		(dnp no)
-		(property "Reference" "R16"
+		(property "Reference" "R12"
 			(at 133.35 73.9139 0)
 			(effects
@@
 			(project "ZEReader-Pico"
 				(path "/ec954637-2a8b-4662-b4a1-f88107f11cb0/5fd074b7-3c47-4717-bcdc-b0d8134ff74e"
-					(reference "R16")
+					(reference "R12")
 					(unit 1)
 				)
@@
 		(on_board yes)
 		(dnp no)
-		(property "Reference" "R12"
+		(property "Reference" "R13"
 			(at 99.06 73.914 0)
 			(effects
@@
 			(project "ZEReader-Pico"
 				(path "/ec954637-2a8b-4662-b4a1-f88107f11cb0/5fd074b7-3c47-4717-bcdc-b0d8134ff74e"
-					(reference "R12")
+					(reference "R13")
 					(unit 1)
 				)
@@
 		(on_board yes)
 		(dnp no)
-		(property "Reference" "R15"
+		(property "Reference" "R16"
 			(at 125.73 73.9139 0)
 			(effects
@@
 			(project "ZEReader-Pico"
 				(path "/ec954637-2a8b-4662-b4a1-f88107f11cb0/5fd074b7-3c47-4717-bcdc-b0d8134ff74e"
-					(reference "R15")
+					(reference "R16")
 					(unit 1)
 				)
@@
 		(on_board yes)
 		(dnp no)
-		(property "Reference" "R14"
+		(property "Reference" "R15"
 			(at 140.97 73.9139 0)
 			(effects
@@
 			(project "ZEReader-Pico"
 				(path "/ec954637-2a8b-4662-b4a1-f88107f11cb0/5fd074b7-3c47-4717-bcdc-b0d8134ff74e"
-					(reference "R14")
+					(reference "R15")
 					(unit 1)
 				)
@@
 		(on_board yes)
 		(dnp no)
-		(property "Reference" "R13"
+		(property "Reference" "R14"
 			(at 102.87 73.914 0)
 			(effects
@@
 			(project ""
 				(path "/ec954637-2a8b-4662-b4a1-f88107f11cb0/5fd074b7-3c47-4717-bcdc-b0d8134ff74e"
-					(reference "R13")
-					(unit 1)
-				)
+					(reference "R14")
+					(unit 1)
+				)

Commit message: Connect both USB data lines again, checked everything with datasheets again
Parts:
- renumbered J6 to J7, R13 to R12, R14 to R13, R17 to R14, R16 to R15, R12 to R16, R15 to R17
Changed lines of the file:
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@@
 		(on_board yes)
 		(dnp no)
-		(property "Reference" "R12"
+		(property "Reference" "R16"
 			(at 133.35 73.9139 0)
 			(effects
@@
 			(project "ZEReader-Pico"
 				(path "/ec954637-2a8b-4662-b4a1-f88107f11cb0/5fd074b7-3c47-4717-bcdc-b0d8134ff74e"
-					(reference "R12")
+					(reference "R16")
 					(unit 1)
 				)
@@
 		(on_board yes)
 		(dnp no)
-		(property "Reference" "R13"
+		(property "Reference" "R12"
 			(at 99.06 73.914 0)
 			(effects
@@
 			(project "ZEReader-Pico"
 				(path "/ec954637-2a8b-4662-b4a1-f88107f11cb0/5fd074b7-3c47-4717-bcdc-b0d8134ff74e"
-					(reference "R13")
+					(reference "R12")
 					(unit 1)
 				)
@@
 		(on_board yes)
 		(dnp no)
-		(property "Reference" "R16"
+		(property "Reference" "R15"
 			(at 125.73 73.9139 0)
 			(effects
@@
 			(project "ZEReader-Pico"
 				(path "/ec954637-2a8b-4662-b4a1-f88107f11cb0/5fd074b7-3c47-4717-bcdc-b0d8134ff74e"
-					(reference "R16")
+					(reference "R15")
 					(unit 1)
 				)
@@
 		(dnp no)
 		(fields_autoplaced yes)
-		(property "Reference" "#PWR033"
+		(property "Reference" "#PWR027"
 			(at 85.09 71.12 0)
 			(effects
@@
 			(project ""
 				(path "/ec954637-2a8b-4662-b4a1-f88107f11cb0/5fd074b7-3c47-4717-bcdc-b0d8134ff74e"
-					(reference "#PWR033")
+					(reference "#PWR027")
 					(unit 1)
 				)
@@
 		(on_board yes)
 		(dnp no)
-		(property "Reference" "R17"
+		(property "Reference" "R14"
 			(at 110.49 73.9139 0)
 			(effects
@@
 			(project "ZEReader-Pico"
 				(path "/ec954637-2a8b-4662-b4a1-f88107f11cb0/5fd074b7-3c47-4717-bcdc-b0d8134ff74e"
-					(reference "R17")
+					(reference "R14")
 					(unit 1)
 				)
@@
 		(on_board yes)
 		(dnp no)
-		(property "Reference" "R15"
+		(property "Reference" "R17"
 			(at 140.97 73.9139 0)
 			(effects
@@
 			(project "ZEReader-Pico"
 				(path "/ec954637-2a8b-4662-b4a1-f88107f11cb0/5fd074b7-3c47-4717-bcdc-b0d8134ff74e"
-					(reference "R15")
+					(reference "R17")
 					(unit 1)
 				)
@@
 		(dnp no)
 		(fields_autoplaced yes)
-		(property "Reference" "#PWR04"
+		(property "Reference" "#PWR028"
 			(at 204.47 116.84 0)
 			(effects
@@
 			(project ""
 				(path "/ec954637-2a8b-4662-b4a1-f88107f11cb0/5fd074b7-3c47-4717-bcdc-b0d8134ff74e"
-					(reference "#PWR04")
+					(reference "#PWR028")
 					(unit 1)
 				)
@@
 		(dnp no)
 		(fields_autoplaced yes)
-		(property "Reference" "#PWR01"
+		(property "Reference" "#PWR025"
 			(at 71.12 121.92 0)
 			(effects
@@
 			(project ""
 				(path "/ec954637-2a8b-4662-b4a1-f88107f11cb0/5fd074b7-3c47-4717-bcdc-b0d8134ff74e"
-					(reference "#PWR01")
+					(reference "#PWR025")
 					(unit 1)
 				)
@@
 		(dnp no)
 		(fields_autoplaced yes)
-		(property "Reference" "#PWR02"
+		(property "Reference" "#PWR026"
 			(at 85.09 53.34 0)
 			(effects
@@
 			(project ""
 				(path "/ec954637-2a8b-4662-b4a1-f88107f11cb0/5fd074b7-3c47-4717-bcdc-b0d8134ff74e"
-					(reference "#PWR02")
+					(reference "#PWR026")
 					(unit 1)
 				)
@@
 		(on_board yes)
 		(dnp no)
-		(property "Reference" "R14"
+		(property "Reference" "R13"
 			(at 102.87 73.914 0)
 			(effects
@@
 			(project ""
 				(path "/ec954637-2a8b-4662-b4a1-f88107f11cb0/5fd074b7-3c47-4717-bcdc-b0d8134ff74e"
-					(reference "R14")
+					(reference "R13")
 					(unit 1)
 				)
@@
 		(dnp no)
 		(fields_autoplaced yes)
-		(property "Reference" "J6"
+		(property "Reference" "J7"
 			(at 182.245 76.2 0)
 			(effects
@@
 			(project ""
 				(path "/ec954637-2a8b-4662-b4a1-f88107f11cb0/5fd074b7-3c47-4717-bcdc-b0d8134ff74e"
-					(reference "J6")
-					(unit 1)
-				)
+					(reference "J7")
+					(unit 1)
+				)

Commit message: Reworked the PCB after review
Connections:
- net SD_DET_A is gone; now on net GND: J7.10 (DET_A)
Changed lines of the file:
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@@
+	)
+	(junction
+		(at 71.12 107.95)
+		(diameter 0)
+		(color 0 0 0 0)
 	)
 	(junction
@@
 	(wire
 		(pts
+			(xy 71.12 111.76) (xy 71.12 107.95)
+		)
+		(stroke
+			(width 0)
+			(type default)
+		)
+	)
+	(wire
+		(pts
 			(xy 139.7 71.12) (xy 139.7 67.31)
 		)
@@
 	(wire
 		(pts
-			(xy 71.12 115.57) (xy 71.12 100.33)
-		)
-		(stroke
-			(width 0)
-			(type default)
-		)
-	)
-	(wire
-		(pts
 			(xy 132.08 90.17) (xy 158.75 90.17)
 		)
@@
 	(wire
 		(pts
-			(xy 88.9 107.95) (xy 158.75 107.95)
-		)
-		(stroke
-			(width 0)
-			(type default)
-		)
-	)
-	(wire
-		(pts
 			(xy 109.22 78.74) (xy 109.22 97.79)
 		)
@@
 	(wire
 		(pts
+			(xy 71.12 107.95) (xy 158.75 107.95)
+		)
+		(stroke
+			(width 0)
+			(type default)
+		)
+	)
+	(wire
+		(pts
 			(xy 139.7 87.63) (xy 139.7 78.74)
 		)
@@
 		(pts
 			(xy 93.98 105.41) (xy 158.75 105.41)
+		)
+		(stroke
+			(width 0)
+			(type default)
+		)
+	)
+	(wire
+		(pts
+			(xy 71.12 107.95) (xy 71.12 100.33)
 		)
 		(stroke
@@
 		(shape bidirectional)
 		(at 88.9 105.41 180)
-		(effects
-			(font
-				(size 1.27 1.27)
-			)
-			(justify right)
-		)
-	)
-	(hierarchical_label "SD_DET_A"
-		(shape bidirectional)
-		(at 88.9 107.95 180)
 		(effects
 			(font
@@
 	(symbol
 		(lib_id "power:GND")
-		(at 71.12 115.57 0)
+		(at 71.12 111.76 0)
 		(unit 1)
 		(exclude_from_sim no)
@@
 		(fields_autoplaced yes)
 		(property "Reference" "#PWR025"
-			(at 71.12 121.92 0)
+			(at 71.12 118.11 0)
 			(effects
 				(font
@@
 		)
 		(property "Value" "GND"
-			(at 71.12 120.65 0)
+			(at 71.12 116.84 0)
 			(effects
 				(font
@@
 		)
 		(property "Footprint" ""
-			(at 71.12 115.57 0)
+			(at 71.12 111.76 0)
 			(effects
 				(font
@@
 		)
 		(property "Datasheet" ""
-			(at 71.12 115.57 0)
+			(at 71.12 111.76 0)
 			(effects
 				(font
@@
 		)
 		(property "Description" "Power symbol creates a global label with name \"GND\" , ground"
-			(at 71.12 115.57 0)
-			(effects
-				(font
+			(at 71.12 111.76 0)
+			(effects
+				(font

Commit message: Bigger Zener, improved BoM, general improvements
Parts:
- C14: DigiKey (none) -> 1276-1804-1-ND; Manufacturer PartNo (none) -> CL31B106KAHNNNE
- J7: DigiKey (none) -> HR1964CT-ND; Manufacturer PartNo (none) -> DM3AT-SF-PEJM5
- R12, R13, R14, R15, R16, R17: DigiKey (none) -> 311-10.0KFRCT-ND; Manufacturer PartNo (none) -> RC1206FR-0710KL
