File: 01_mcu.kicad_sch (KiCad schematic)
At the start: 3 parts, among them J1 UART, J2 Conn_02x05_Odd_Even

Commit message: Avoid using the ADC pins for anything but ADC tasks
Connections:
- net CHARGING: now also A1.4 (GPIO2); no longer A1.31 (GPIO26_ADC0)
- net UC_OFF: now also A1.6 (GPIO4); no longer A1.34 (GPIO28_ADC2)
- net UC_ON_OFF_INTERRUPT: now also A1.5 (GPIO3); no longer A1.32 (GPIO27_ADC1)
- no-connect marks 17 -> 14
Other:
- moved on the sheet: J1
Changed lines of the file:
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@@
-	)
-	(no_connect
-		(at 135.89 92.71)
 	)
 	(no_connect
@@
 	)
 	(no_connect
-		(at 135.89 90.17)
-	)
-	(no_connect
 		(at 99.06 64.77)
 	)
@@
 	)
 	(no_connect
-		(at 135.89 87.63)
-	)
-	(no_connect
 		(at 181.61 85.09)
 	)
@@
 	(wire
 		(pts
-			(xy 107.95 87.63) (xy 106.68 87.63)
-		)
-		(stroke
-			(width 0)
-			(type default)
-		)
-	)
-	(wire
-		(pts
-			(xy 106.68 85.09) (xy 135.89 85.09)
+			(xy 96.52 87.63) (xy 95.25 87.63)
+		)
+		(stroke
+			(width 0)
+			(type default)
+		)
+	)
+	(wire
+		(pts
+			(xy 95.25 85.09) (xy 135.89 85.09)
+		)
+		(stroke
+			(width 0)
+			(type default)
+		)
+	)
+	(wire
+		(pts
+			(xy 127 92.71) (xy 135.89 92.71)
 		)
 		(stroke
@@
 	(wire
 		(pts
-			(xy 181.61 115.57) (xy 189.23 115.57)
-		)
-		(stroke
-			(width 0)
-			(type default)
-		)
-	)
-	(wire
-		(pts
 			(xy 92.71 77.47) (xy 92.71 74.93)
 		)
@@
 	(wire
 		(pts
+			(xy 127 90.17) (xy 135.89 90.17)
+		)
+		(stroke
+			(width 0)
+			(type default)
+		)
+	)
+	(wire
+		(pts
 			(xy 127 97.79) (xy 135.89 97.79)
 		)
@@
 	(wire
 		(pts
-			(xy 107.95 91.44) (xy 107.95 87.63)
+			(xy 96.52 91.44) (xy 96.52 87.63)
 		)
 		(stroke
@@
 	(wire
 		(pts
-			(xy 181.61 110.49) (xy 189.23 110.49)
-		)
-		(stroke
-			(width 0)
-			(type default)
-		)
-	)
-	(wire
-		(pts
-			(xy 181.61 113.03) (xy 189.23 113.03)
-		)
-		(stroke
-			(width 0)
-			(type default)
-		)
-	)
-	(wire
-		(pts
 			(xy 127 110.49) (xy 135.89 110.49)
 		)
@@
 	(wire
 		(pts
-			(xy 106.68 82.55) (xy 135.89 82.55)
+			(xy 95.25 82.55) (xy 135.89 82.55)
 		)
 		(stroke
@@
 		(pts
 			(xy 127 113.03) (xy 135.89 113.03)
+		)
+		(stroke
+			(width 0)
+			(type default)
+		)
+	)
+	(wire
+		(pts
+			(xy 127 87.63) (xy 135.89 87.63)
 		)
 		(stroke
@@
 	(hierarchical_label "UC_OFF"
 		(shape output)
-		(at 189.23 115.57 0)
-		(effects
-			(font
-				(size 1.27 1.27)
-			)
-			(justify left)
+		(at 127 92.71 180)
+		(effects
+			(font
+				(size 1.27 1.27)
+			)
+			(justify right)
 		)
 	)
 	(hierarchical_label "UC_ON_OFF_INTERRUPT"
 		(shape input)
-		(at 189.23 113.03 0)
-		(effects
-			(font
-				(size 1.27 1.27)
-			)
-			(justify left)
+		(at 127 90.17 180)
+		(effects
+			(font
+				(size 1.27 1.27)
+			)
+			(justify right)
 		)
 	)
@@
 	(hierarchical_label "CHARGING"
 		(shape input)
-		(at 189.23 110.49 0)
-		(effects
-			(font
-				(size 1.27 1.27)
-			)
-			(justify left)
+		(at 127 87.63 180)
+		(effects
+			(font
+				(size 1.27 1.27)
+			)
+			(justify right)
 		)
 	)
@@
 	(symbol
 		(lib_id "Connector:Conn_01x03_Pin")
-		(at 101.6 85.09 0)
+		(at 90.17 85.09 0)
 		(mirror x)
 		(unit 1)
@@
 		(dnp no)
 		(property "Reference" "J1"
-			(at 98.044 87.376 0)
+			(at 86.614 87.376 0)
 			(effects
 				(font
@@
 		)
 		(property "Value" "UART"
-			(at 98.044 85.09 0)
+			(at 86.614 85.09 0)
 			(effects
 				(font
@@
 		)
 		(property "Footprint" "Connector_PinHeader_2.54mm:PinHeader_1x03_P2.54mm_Vertical"
-			(at 101.6 85.09 0)
+			(at 90.17 85.09 0)
 			(effects
 				(font
@@
 		)
 		(property "Datasheet" "https://cdn.amphenol-cs.com/media/wysiwyg/files/documentation/datasheet/boardwiretoboard/bwb_agilbrick_2_54mm_btb_header_g800.pdf"
-			(at 101.6 85.09 0)
+			(at 90.17 85.09 0)
 			(effects
 				(font
@@
 		)
 		(property "Description" "Steckverbinder Steckleiste Durchkontaktierung 3 positionen 0,100\" (2,54mm)"
-			(at 101.6 85.09 0)
+			(at 90.17 85.09 0)
 			(effects
 				(font
@@
 		)
 		(property "DATASHEET-URL" ""
-			(at 101.6 85.09 0)
+			(at 90.17 85.09 0)
 			(effects
 				(font
@@
 		)
 		(property "DigiKey" "664-G800W305018EU-ND"
-			(at 101.6 85.09 0)
+			(at 90.17 85.09 0)
 			(effects
 				(font
@@
 		)
 		(property "IR" ""
-			(at 101.6 85.09 0)
+			(at 90.17 85.09 0)
 			(effects
 				(font
@@
 		)
 		(property "Manufacturer PartNo" "G800W305018EU"
-			(at 101.6 85.09 0)
+			(at 90.17 85.09 0)
 			(effects
 				(font
@@
 		)
 		(property "PACKAGING" ""
-			(at 101.6 85.09 0)
+			(at 90.17 85.09 0)
 			(effects
 				(font
@@
 		)
 		(property "PART-NUMBER" ""
-			(at 101.6 85.09 0)
+			(at 90.17 85.09 0)
 			(effects
 				(font
@@
 		)
 		(property "QTY" ""
-			(at 101.6 85.09 0)
+			(at 90.17 85.09 0)
 			(effects
 				(font
@@
 		)
 		(property "VR" ""
-			(at 101.6 85.09 0)
+			(at 90.17 85.09 0)
 			(effects
 				(font
@@
 	(symbol
 		(lib_id "power:GND")
-		(at 107.95 91.44 0)
+		(at 96.52 91.44 0)
 		(unit 1)
 		(exclude_from_sim no)
@@
 		(fields_autoplaced yes)
 		(property "Reference" "#PWR06"
-			(at 107.95 97.79 0)
+			(at 96.52 97.79 0)
 			(effects
 				(font
@@
 		)
 		(property "Value" "GND"
-			(at 107.95 96.52 0)
+			(at 96.52 96.52 0)
 			(effects
 				(font
@@
 		)
 		(property "Footprint" ""
-			(at 107.95 91.44 0)
+			(at 96.52 91.44 0)
 			(effects
 				(font
@@
 		)
 		(property "Datasheet" ""
-			(at 107.95 91.44 0)
+			(at 96.52 91.44 0)
 			(effects
 				(font
@@
 		)
 		(property "Description" "Power symbol creates a global label with name \"GND\" , ground"
-			(at 107.95 91.44 0)
-			(effects
-				(font
+			(at 96.52 91.44 0)
+			(effects
+				(font

Commit message: Add an voltage bypass mode when USB-C is connected
When USB-C is connected, the device should be charging, but also powered,
without taking care of the on/off button's state.
Otherwise, flashing the device via USB-C would only be
possible as long as the button is pressed which makes the usage
experience a mess and flaky.
This uses p-MOSFETs to do the switch and
a) avoid a battery voltage going to the system when USB-C is connected
b) avoid powering having both, USB-C and Micro-USB active

TODO: This adds the basic idea, routing must be fixed!
Connections:
- no-connect marks 14 -> 17
Changed lines of the file:
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@@
+	)
+	(no_connect
+		(at 181.61 113.03)
 	)
 	(no_connect
@@
 	)
 	(no_connect
+		(at 181.61 115.57)
+	)
+	(no_connect
+		(at 181.61 110.49)
+	)
+	(no_connect
