File: 03_epaper-driver.kicad_sch (KiCad schematic)
At the start: 21 parts, among them J7 FFC2B28-24-G, Q1 BSS138

Commit message: Reworked v2 routing
- some general improvements
- reworked component numbering
- routed and tuned differential pair (USB)
- added stiching vias and improved ground fills
Parts:
- renumbered C10 to C11, C11 to C12, C5 to C13, C2 to C4, C4 to C5, C7 to C6, C6 to C7, D2 to D5, D3 to D6, D1 to D7, Drain1 to DRAIN1, J7 to J2, Q1 to Q3, R9 to R7
Changed lines of the file:
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@@
+	(wire
+		(pts
+			(xy 176.53 53.34) (xy 176.53 83.82)
+		)
+		(stroke
+			(width 0)
+			(type default)
+		)
+	)
 	(wire
 		(pts
@@
 		(on_board yes)
 		(dnp no)
-		(property "Reference" "C10"
+		(property "Reference" "C11"
 			(at 155.956 67.564 90)
 			(effects
@@
 			(project "ZEReader-Pico"
 				(path "/ec954637-2a8b-4662-b4a1-f88107f11cb0/d006ff72-e176-4e99-8906-01d59b86077c"
-					(reference "C10")
+					(reference "C11")
 					(unit 1)
 				)
@@
 	(symbol
 		(lib_id "power:+3.3V")
-		(at 176.53 83.82 90)
+		(at 176.53 53.34 0)
 		(unit 1)
 		(exclude_from_sim no)
@@
 		(dnp no)
 		(property "Reference" "#PWR013"
-			(at 180.34 83.82 0)
+			(at 176.53 57.15 0)
 			(effects
 				(font
@@
 		)
 		(property "Value" "+3.3V"
-			(at 179.324 82.804 90)
+			(at 179.832 53.086 0)
 			(effects
 				(font
@@
 		)
 		(property "Footprint" ""
-			(at 176.53 83.82 0)
+			(at 176.53 53.34 0)
 			(effects
 				(font
@@
 		)
 		(property "Datasheet" ""
-			(at 176.53 83.82 0)
+			(at 176.53 53.34 0)
 			(effects
 				(font
@@
 		)
 		(property "Description" "Power symbol creates a global label with name \"+3.3V\""
-			(at 176.53 83.82 0)
+			(at 176.53 53.34 0)
 			(effects
 				(font
@@
 		(dnp no)
 		(fields_autoplaced yes)
-		(property "Reference" "C2"
+		(property "Reference" "C4"
 			(at 41.91 82.5499 0)
 			(effects
@@
 			(project ""
 				(path "/ec954637-2a8b-4662-b4a1-f88107f11cb0/d006ff72-e176-4e99-8906-01d59b86077c"
-					(reference "C2")
+					(reference "C4")
 					(unit 1)
 				)
@@
 		(dnp no)
 		(fields_autoplaced yes)
-		(property "Reference" "D3"
+		(property "Reference" "D6"
 			(at 95.5675 69.85 0)
 			(effects
@@
 			(project ""
 				(path "/ec954637-2a8b-4662-b4a1-f88107f11cb0/d006ff72-e176-4e99-8906-01d59b86077c"
-					(reference "D3")
+					(reference "D6")
 					(unit 1)
 				)
@@
 		(on_board yes)
 		(dnp no)
-		(property "Reference" "J7"
+		(property "Reference" "J2"
 			(at 203.454 56.642 0)
 			(effects
@@
 			(project ""
 				(path "/ec954637-2a8b-4662-b4a1-f88107f11cb0/d006ff72-e176-4e99-8906-01d59b86077c"
-					(reference "J7")
+					(reference "J2")
 					(unit 1)
 				)
@@
 		(on_board yes)
 		(dnp no)
-		(property "Reference" "C7"
+		(property "Reference" "C6"
 			(at 155.448 85.344 90)
 			(effects
@@
 			(project "ZEReader-Pico"
 				(path "/ec954637-2a8b-4662-b4a1-f88107f11cb0/d006ff72-e176-4e99-8906-01d59b86077c"
-					(reference "C7")
+					(reference "C6")
 					(unit 1)
 				)
@@
 		(on_board yes)
 		(dnp no)
-		(property "Reference" "C5"
+		(property "Reference" "C13"
 			(at 120.65 91.948 90)
 			(effects
@@
 			(project "ZEReader-Pico"
 				(path "/ec954637-2a8b-4662-b4a1-f88107f11cb0/d006ff72-e176-4e99-8906-01d59b86077c"
-					(reference "C5")
+					(reference "C13")
 					(unit 1)
 				)
@@
 		(dnp no)
 		(fields_autoplaced yes)
-		(property "Reference" "R9"
+		(property "Reference" "R7"
 			(at 66.04 110.4899 0)
 			(effects
@@
 			(project "ZEReader-Pico"
 				(path "/ec954637-2a8b-4662-b4a1-f88107f11cb0/d006ff72-e176-4e99-8906-01d59b86077c"
-					(reference "R9")
+					(reference "R7")
 					(unit 1)
 				)
@@
 		(on_board yes)
 		(dnp no)
-		(property "Reference" "C11"
+		(property "Reference" "C12"
 			(at 155.956 62.484 90)
 			(effects
@@
 			(project "ZEReader-Pico"
 				(path "/ec954637-2a8b-4662-b4a1-f88107f11cb0/d006ff72-e176-4e99-8906-01d59b86077c"
-					(reference "C11")
+					(reference "C12")
 					(unit 1)
 				)
@@
 		(on_board yes)
 		(dnp no)
-		(property "Reference" "C6"
+		(property "Reference" "C7"
 			(at 155.448 110.744 90)
 			(effects
@@
 			(project ""
 				(path "/ec954637-2a8b-4662-b4a1-f88107f11cb0/d006ff72-e176-4e99-8906-01d59b86077c"
-					(reference "C6")
+					(reference "C7")
 					(unit 1)
 				)
@@
 		(on_board yes)
 		(dnp no)
-		(property "Reference" "D2"
+		(property "Reference" "D5"
 			(at 96.52 92.456 0)
 			(effects
@@
 			(project ""
 				(path "/ec954637-2a8b-4662-b4a1-f88107f11cb0/d006ff72-e176-4e99-8906-01d59b86077c"
-					(reference "D2")
+					(reference "D5")
 					(unit 1)
 				)
@@
 		(dnp no)
 		(fields_autoplaced yes)
-		(property "Reference" "Q1"
+		(property "Reference" "Q3"
 			(at 67.31 91.4399 0)
 			(effects
@@
 			(project ""
 				(path "/ec954637-2a8b-4662-b4a1-f88107f11cb0/d006ff72-e176-4e99-8906-01d59b86077c"
-					(reference "Q1")
+					(reference "Q3")
 					(unit 1)
 				)
@@
 		(dnp no)
 		(fields_autoplaced yes)
-		(property "Reference" "D1"
+		(property "Reference" "D7"
 			(at 96.8375 113.03 0)
 			(effects
@@
 			(project ""
 				(path "/ec954637-2a8b-4662-b4a1-f88107f11cb0/d006ff72-e176-4e99-8906-01d59b86077c"
-					(reference "D1")
+					(reference "D7")
 					(unit 1)
 				)
@@
 		(on_board yes)
 		(dnp no)
-		(property "Reference" "C4"
+		(property "Reference" "C5"
 			(at 120.65 70.104 90)
 			(effects
@@
 			(project "ZEReader-Pico"
 				(path "/ec954637-2a8b-4662-b4a1-f88107f11cb0/d006ff72-e176-4e99-8906-01d59b86077c"
-					(reference "C4")
+					(reference "C5")
 					(unit 1)
 				)
@@
 		(on_board yes)
 		(dnp no)
-		(property "Reference" "Drain1"
+		(property "Reference" "DRAIN1"
 			(at 51.562 173.736 90)
 			(effects
@@
 			(project "ZEReader-Pico"
 				(path "/ec954637-2a8b-4662-b4a1-f88107f11cb0/d006ff72-e176-4e99-8906-01d59b86077c"
-					(reference "Drain1")
+					(reference "DRAIN1")
 					(unit 1)
 				)

Commit message: some minor improvements after evaluating the CI run
Parts:
- C11, C13, C5, C7, C9: value 1uF/25V -> 1uF, 25V
- C12: value 1uF/50V -> 1uF, 50V
- C6: value 10uF/10V -> 10uF, 10V
- C8: value 1uF/10V -> 1uF, 10V
- DRAIN1, G/GDR1, S/RESE1: now left out of the parts list
Changed lines of the file:
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@@
 		(title "ZEReader-Pico")
 		(date "{kibot_date}")
-		(rev "v1")
+		(rev "v2")
 		(company "Anna-Lena Marx")
 		(comment 4 "Git revision: {kibot_git-hash}")
@@
 			)
 		)
-		(property "Value" "1uF/25V"
+		(property "Value" "1uF, 25V"
 			(at 163.322 67.564 90)
 			(effects
@@
 			)
 		)
-		(property "Value" "1uF/10V"
+		(property "Value" "1uF, 10V"
 			(at 163.576 77.724 90)
 			(effects
@@
 			)
 		)
-		(property "Value" "10uF/10V"
+		(property "Value" "10uF, 10V"
 			(at 163.068 85.344 90)
 			(effects
@@
 			)
 		)
-		(property "Value" "1uF/25V"
+		(property "Value" "1uF, 25V"
 			(at 120.65 94.234 90)
 			(effects
@@
 			)
 		)
-		(property "Value" "1uF/50V"
+		(property "Value" "1uF, 50V"
 			(at 163.322 62.484 90)
 			(effects
@@
 			)
 		)
-		(property "Value" "1uF/25V"
+		(property "Value" "1uF, 25V"
 			(at 163.322 110.744 90)
 			(effects
@@
 			)
 		)
-		(property "Value" "1uF/25V"
+		(property "Value" "1uF, 25V"
 			(at 120.65 72.136 90)
 			(effects
@@
 		(unit 1)
 		(exclude_from_sim no)
-		(in_bom yes)
+		(in_bom no)
 		(on_board yes)
 		(dnp no)
@@
 		(unit 1)
 		(exclude_from_sim no)
-		(in_bom yes)
+		(in_bom no)
 		(on_board yes)
 		(dnp no)
@@
 		(unit 1)
 		(exclude_from_sim no)
-		(in_bom yes)
+		(in_bom no)
 		(on_board yes)
 		(dnp no)
@@
 			)
 		)
-		(property "Value" "1uF/25V"
+		(property "Value" "1uF, 25V"
 			(at 163.322 72.644 90)
 			(effects

Commit message: v2: final touch
- add proper ESD diodes for USB
- move the USB fuse right after the connector
- pretty labels for test points
Parts:
- renumbered C9 to C5, C8 to C6, C5 to C7, C7 to C8, C6 to C9, D5 to D4, D7 to D5, R8 to R7, R7 to R8
Changed lines of the file:
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@@
 		(on_board yes)
 		(dnp no)
-		(property "Reference" "C8"
+		(property "Reference" "C6"
 			(at 155.448 77.724 90)
 			(effects
@@
 			(project "ZEReader-Pico"
 				(path "/ec954637-2a8b-4662-b4a1-f88107f11cb0/d006ff72-e176-4e99-8906-01d59b86077c"
-					(reference "C8")
+					(reference "C6")
 					(unit 1)
 				)
@@
 		(on_board yes)
 		(dnp no)
-		(property "Reference" "C6"
+		(property "Reference" "C9"
 			(at 155.448 85.344 90)
 			(effects
@@
 			(project "ZEReader-Pico"
 				(path "/ec954637-2a8b-4662-b4a1-f88107f11cb0/d006ff72-e176-4e99-8906-01d59b86077c"
-					(reference "C6")
+					(reference "C9")
 					(unit 1)
 				)
@@
 		(on_board yes)
 		(dnp no)
-		(property "Reference" "R8"
+		(property "Reference" "R7"
 			(at 53.34 110.4899 0)
 			(effects
@@
 			(project ""
 				(path "/ec954637-2a8b-4662-b4a1-f88107f11cb0/d006ff72-e176-4e99-8906-01d59b86077c"
-					(reference "R8")
+					(reference "R7")
 					(unit 1)
 				)
@@
 		(dnp no)
 		(fields_autoplaced yes)
-		(property "Reference" "R7"
+		(property "Reference" "R8"
 			(at 66.04 110.4899 0)
 			(effects
@@
 			(project "ZEReader-Pico"
 				(path "/ec954637-2a8b-4662-b4a1-f88107f11cb0/d006ff72-e176-4e99-8906-01d59b86077c"
-					(reference "R7")
+					(reference "R8")
 					(unit 1)
 				)
@@
 		(on_board yes)
 		(dnp no)
-		(property "Reference" "C7"
+		(property "Reference" "C8"
 			(at 155.448 110.744 90)
 			(effects
@@
 			(project ""
 				(path "/ec954637-2a8b-4662-b4a1-f88107f11cb0/d006ff72-e176-4e99-8906-01d59b86077c"
-					(reference "C7")
+					(reference "C8")
 					(unit 1)
 				)
@@
 		(on_board yes)
 		(dnp no)
-		(property "Reference" "D5"
+		(property "Reference" "D4"
 			(at 96.52 92.456 0)
 			(effects
@@
 			(project ""
 				(path "/ec954637-2a8b-4662-b4a1-f88107f11cb0/d006ff72-e176-4e99-8906-01d59b86077c"
-					(reference "D5")
+					(reference "D4")
 					(unit 1)
 				)
@@
 		(dnp no)
 		(fields_autoplaced yes)
-		(property "Reference" "D7"
+		(property "Reference" "D5"
 			(at 96.8375 113.03 0)
 			(effects
@@
 			(project ""
 				(path "/ec954637-2a8b-4662-b4a1-f88107f11cb0/d006ff72-e176-4e99-8906-01d59b86077c"
-					(reference "D7")
+					(reference "D5")
 					(unit 1)
 				)
@@
 		(on_board yes)
 		(dnp no)
-		(property "Reference" "C5"
+		(property "Reference" "C7"
 			(at 120.65 70.104 90)
 			(effects
@@
 			(project "ZEReader-Pico"
 				(path "/ec954637-2a8b-4662-b4a1-f88107f11cb0/d006ff72-e176-4e99-8906-01d59b86077c"
-					(reference "C5")
+					(reference "C7")
 					(unit 1)
 				)
@@
 		(on_board yes)
 		(dnp no)
-		(property "Reference" "C9"
+		(property "Reference" "C5"
 			(at 155.448 72.644 90)
 			(effects
@@
 			(project "ZEReader-Pico"
 				(path "/ec954637-2a8b-4662-b4a1-f88107f11cb0/d006ff72-e176-4e99-8906-01d59b86077c"
-					(reference "C9")
-					(unit 1)
-				)
+					(reference "C5")
+					(unit 1)
+				)

Commit message: Connect both USB data lines again, checked everything with datasheets again
Parts:
- renumbered C5 to C10, C6 to C11, C9 to C12, C8 to C13, C3 to C5, C7 to C6, C13 to C7, C12 to C8, C11 to C9, D6 to D7, D4 to D8, D5 to D9, J2 to J6, Q3 to Q4, R7 to R10, R8 to R11
Changed lines of the file:
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@@
 		(on_board yes)
 		(dnp no)
-		(property "Reference" "C11"
+		(property "Reference" "C9"
 			(at 155.956 67.564 90)
 			(effects
@@
 			(project "ZEReader-Pico"
 				(path "/ec954637-2a8b-4662-b4a1-f88107f11cb0/d006ff72-e176-4e99-8906-01d59b86077c"
-					(reference "C11")
+					(reference "C9")
 					(unit 1)
 				)
@@
 		(on_board yes)
 		(dnp no)
-		(property "Reference" "#PWR013"
+		(property "Reference" "#PWR023"
 			(at 176.53 57.15 0)
 			(effects
@@
 			(project ""
 				(path "/ec954637-2a8b-4662-b4a1-f88107f11cb0/d006ff72-e176-4e99-8906-01d59b86077c"
-					(reference "#PWR013")
+					(reference "#PWR023")
 					(unit 1)
 				)
@@
 		(on_board yes)
 		(dnp no)
-		(property "Reference" "C6"
+		(property "Reference" "C11"
 			(at 155.448 77.724 90)
 			(effects
@@
 			(project "ZEReader-Pico"
 				(path "/ec954637-2a8b-4662-b4a1-f88107f11cb0/d006ff72-e176-4e99-8906-01d59b86077c"
-					(reference "C6")
+					(reference "C11")
 					(unit 1)
 				)
@@
 		(on_board yes)
 		(dnp no)
-		(property "Reference" "C3"
+		(property "Reference" "C5"
 			(at 87.63 86.3599 0)
 			(effects
@@
 			(project "ZEReader-Pico"
 				(path "/ec954637-2a8b-4662-b4a1-f88107f11cb0/d006ff72-e176-4e99-8906-01d59b86077c"
-					(reference "C3")
+					(reference "C5")
 					(unit 1)
 				)
@@
 		(dnp no)
 		(fields_autoplaced yes)
-		(property "Reference" "D6"
+		(property "Reference" "D7"
 			(at 95.5675 69.85 0)
 			(effects
@@
 			(project ""
 				(path "/ec954637-2a8b-4662-b4a1-f88107f11cb0/d006ff72-e176-4e99-8906-01d59b86077c"
-					(reference "D6")
+					(reference "D7")
 					(unit 1)
 				)
@@
 		(on_board yes)
 		(dnp no)
-		(property "Reference" "J2"
+		(property "Reference" "J6"
 			(at 203.454 56.642 0)
 			(effects
@@
 			(project ""
 				(path "/ec954637-2a8b-4662-b4a1-f88107f11cb0/d006ff72-e176-4e99-8906-01d59b86077c"
-					(reference "J2")
+					(reference "J6")
 					(unit 1)
 				)
@@
 		(dnp no)
 		(fields_autoplaced yes)
-		(property "Reference" "#PWR010"
+		(property "Reference" "#PWR021"
 			(at 128.27 127 0)
 			(effects
@@
 			(project "ZEReader-Pico"
 				(path "/ec954637-2a8b-4662-b4a1-f88107f11cb0/d006ff72-e176-4e99-8906-01d59b86077c"
-					(reference "#PWR010")
+					(reference "#PWR021")
 					(unit 1)
 				)
@@
 		(on_board yes)
 		(dnp no)
-		(property "Reference" "C9"
+		(property "Reference" "C12"
 			(at 155.448 85.344 90)
 			(effects
@@
 			(project "ZEReader-Pico"
 				(path "/ec954637-2a8b-4662-b4a1-f88107f11cb0/d006ff72-e176-4e99-8906-01d59b86077c"
-					(reference "C9")
+					(reference "C12")
 					(unit 1)
 				)
@@
 		(on_board yes)
 		(dnp no)
-		(property "Reference" "R7"
+		(property "Reference" "R10"
 			(at 53.34 110.4899 0)
 			(effects
@@
 			(project ""
 				(path "/ec954637-2a8b-4662-b4a1-f88107f11cb0/d006ff72-e176-4e99-8906-01d59b86077c"
-					(reference "R7")
+					(reference "R10")
 					(unit 1)
 				)
@@
 		(on_board yes)
 		(dnp no)
-		(property "Reference" "#PWR03"
+		(property "Reference" "#PWR024"
 			(at 191.77 140.97 0)
 			(effects
@@
 			(project ""
 				(path "/ec954637-2a8b-4662-b4a1-f88107f11cb0/d006ff72-e176-4e99-8906-01d59b86077c"
-					(reference "#PWR03")
+					(reference "#PWR024")
 					(unit 1)
 				)
@@
 		(on_board yes)
 		(dnp no)
-		(property "Reference" "C13"
+		(property "Reference" "C7"
 			(at 120.65 91.948 90)
 			(effects
@@
 			(project "ZEReader-Pico"
 				(path "/ec954637-2a8b-4662-b4a1-f88107f11cb0/d006ff72-e176-4e99-8906-01d59b86077c"
-					(reference "C13")
+					(reference "C7")
 					(unit 1)
 				)
@@
 		(dnp no)
 		(fields_autoplaced yes)
-		(property "Reference" "R8"
+		(property "Reference" "R11"
 			(at 66.04 110.4899 0)
 			(effects
@@
 			(project "ZEReader-Pico"
 				(path "/ec954637-2a8b-4662-b4a1-f88107f11cb0/d006ff72-e176-4e99-8906-01d59b86077c"
-					(reference "R8")
+					(reference "R11")
 					(unit 1)
 				)
@@
 		(on_board yes)
 		(dnp no)
-		(property "Reference" "C12"
+		(property "Reference" "C8"
 			(at 155.956 62.484 90)
 			(effects
@@
 			(project "ZEReader-Pico"
 				(path "/ec954637-2a8b-4662-b4a1-f88107f11cb0/d006ff72-e176-4e99-8906-01d59b86077c"
-					(reference "C12")
+					(reference "C8")
 					(unit 1)
 				)
@@
 		(dnp no)
 		(fields_autoplaced yes)
-		(property "Reference" "#PWR08"
+		(property "Reference" "#PWR018"
 			(at 38.1 69.85 0)
 			(effects
@@
 			(project ""
 				(path "/ec954637-2a8b-4662-b4a1-f88107f11cb0/d006ff72-e176-4e99-8906-01d59b86077c"
-					(reference "#PWR08")
+					(reference "#PWR018")
 					(unit 1)
 				)
@@
 		(on_board yes)
 		(dnp no)
-		(property "Reference" "C8"
+		(property "Reference" "C13"
 			(at 155.448 110.744 90)
 			(effects
@@
 			(project ""
 				(path "/ec954637-2a8b-4662-b4a1-f88107f11cb0/d006ff72-e176-4e99-8906-01d59b86077c"
-					(reference "C8")
+					(reference "C13")
 					(unit 1)
 				)
@@
 		(dnp no)
 		(fields_autoplaced yes)
-		(property "Reference" "#PWR011"
+		(property "Reference" "#PWR022"
 			(at 152.4 133.35 0)
 			(effects
@@
 			(project "ZEReader-Pico"
 				(path "/ec954637-2a8b-4662-b4a1-f88107f11cb0/d006ff72-e176-4e99-8906-01d59b86077c"
-					(reference "#PWR011")
+					(reference "#PWR022")
 					(unit 1)
 				)
@@
 		(on_board yes)
 		(dnp no)
-		(property "Reference" "D4"
+		(property "Reference" "D8"
 			(at 96.52 92.456 0)
 			(effects
@@
 			(project ""
 				(path "/ec954637-2a8b-4662-b4a1-f88107f11cb0/d006ff72-e176-4e99-8906-01d59b86077c"
-					(reference "D4")
+					(reference "D8")
 					(unit 1)
 				)
@@
 		(dnp no)
 		(fields_autoplaced yes)
-		(property "Reference" "Q3"
+		(property "Reference" "Q4"
 			(at 67.31 91.4399 0)
 			(effects
@@
 			(project ""
 				(path "/ec954637-2a8b-4662-b4a1-f88107f11cb0/d006ff72-e176-4e99-8906-01d59b86077c"
-					(reference "Q3")
+					(reference "Q4")
 					(unit 1)
 				)
@@
 		(dnp no)
 		(fields_autoplaced yes)
-		(property "Reference" "D5"
+		(property "Reference" "D9"
 			(at 96.8375 113.03 0)
 			(effects
@@
 			(project ""
 				(path "/ec954637-2a8b-4662-b4a1-f88107f11cb0/d006ff72-e176-4e99-8906-01d59b86077c"
-					(reference "D5")
+					(reference "D9")
 					(unit 1)
 				)
@@
 		(on_board yes)
 		(dnp no)
-		(property "Reference" "C7"
+		(property "Reference" "C6"
 			(at 120.65 70.104 90)
 			(effects
@@
 			(project "ZEReader-Pico"
 				(path "/ec954637-2a8b-4662-b4a1-f88107f11cb0/d006ff72-e176-4e99-8906-01d59b86077c"
-					(reference "C7")
+					(reference "C6")
 					(unit 1)
 				)
@@
 		(on_board yes)
 		(dnp no)
-		(property "Reference" "C5"
+		(property "Reference" "C10"
 			(at 155.448 72.644 90)
 			(effects
@@
 			(project "ZEReader-Pico"
 				(path "/ec954637-2a8b-4662-b4a1-f88107f11cb0/d006ff72-e176-4e99-8906-01d59b86077c"
-					(reference "C5")
+					(reference "C10")
 					(unit 1)
 				)
@@
 		(dnp no)
 		(fields_autoplaced yes)
-		(property "Reference" "#PWR07"
+		(property "Reference" "#PWR020"
 			(at 63.5 125.73 0)
 			(effects
@@
 			(project "ZEReader-Pico"
 				(path "/ec954637-2a8b-4662-b4a1-f88107f11cb0/d006ff72-e176-4e99-8906-01d59b86077c"
-					(reference "#PWR07")
+					(reference "#PWR020")
 					(unit 1)
 				)
@@
 		(dnp no)
 		(fields_autoplaced yes)
-		(property "Reference" "#PWR09"
+		(property "Reference" "#PWR019"
 			(at 49.53 125.73 0)
 			(effects
@@
 			(project "ZEReader-Pico"
 				(path "/ec954637-2a8b-4662-b4a1-f88107f11cb0/d006ff72-e176-4e99-8906-01d59b86077c"
-					(reference "#PWR09")
-					(unit 1)
-				)
+					(reference "#PWR019")
+					(unit 1)
+				)

Commit message: Reworked the PCB after review
Changed lines of the file:
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@@
+		)
+	)
+	(text_box "https://files.waveshare.com/upload/8/8e/E-Paper_Driver_HAT.pdf"
+		(exclude_from_sim no)
+		(at 12.7 16.51 0)
+		(size 127 3.81)
+		(margins 0.9525 0.9525 0.9525 0.9525)
+		(stroke
+			(width 0)
+			(type solid)
+		)
+		(fill
+			(type none)
+		)
+		(effects
+			(font
+				(size 1.27 1.27)
+			)
+			(justify left top)
+			(href "https://files.waveshare.com/upload/8/8e/E-Paper_Driver_HAT.pdf")
 		)
 	)
@@
 		)
 	)
+	(text_box "https://v4.cecdn.yun300.cn/100001_1909185148/GDEY075T7.pdf -> Reference Circuit S. 40"
+		(exclude_from_sim no)
+		(at 12.7 20.32 0)
+		(size 127 3.81)
+		(margins 0.9525 0.9525 0.9525 0.9525)
+		(stroke
+			(width 0)
+			(type solid)
+		)
+		(fill
+			(type none)
+		)
+		(effects
+			(font
+				(size 1.27 1.27)
+			)
+			(justify left top)
+			(href "https://v4.cecdn.yun300.cn/100001_1909185148/GDEY075T7.pdf")
+		)
+	)
 	(text_box "Needs testing on the finished PCB if 4.7uF or 10uF"
 		(exclude_from_sim no)
 		(at 15.24 82.55 0)
 		(size 17.78 8.89)
+		(margins 0.9525 0.9525 0.9525 0.9525)
+		(stroke
+			(width 0)
+			(type solid)
+		)
+		(fill
+			(type none)
+		)
+		(effects
+			(font
+				(size 1.27 1.27)
+			)
+			(justify left top)
+		)
+	)
+	(text_box "https://www.buydisplay.com/download/ic/UC8179.pdf?srsltid=AfmBOorGWKpt56S8v_SEIg68MTf0PBAwJ0nzrTD0Z42XBr54EIzW-IkT (Controller itself, S.55)"
+		(exclude_from_sim no)
+		(at 12.7 24.13 0)
+		(size 127 3.81)
 		(margins 0.9525 0.9525 0.9525 0.9525)
 		(stroke
@@
 		)
 	)
-	(text_box "Reference:\nhttps://files.waveshare.com/upload/8/8e/E-Paper_Driver_HAT.pdf\nhttps://v4.cecdn.yun300.cn/100001_1909185148/GDEY075T7.pdf -> Reference Circuit S. 40\nhttps://www.buydisplay.com/download/ic/UC8179.pdf?srsltid=AfmBOorGWKpt56S8v_SEIg68MTf0PBAwJ0nzrTD0Z42XBr54EIzW-IkT (Controller itself, S.55)\n\nnot needed:\n- RPI GPIO Header\n- 9 Pin Header\n- Switch 3/4 line SPI -> connect and use 4 line SPI\n- Level Shifting (TXB0108E), 3.3V used due to RP2350\n- Regulator (RT9193-33) \n	-> the breakout is intended for use with 3.3V and 5V (not needed here)"
+	(text_box "Reference:\n\n\n\n\n\n\n\n\nnot needed:\n- RPI GPIO Header\n- 9 Pin Header\n- Switch 3/4 line SPI -> connect and use 4 line SPI\n- Level Shifting (TXB0108E), 3.3V used due to RP2350\n- Regulator (RT9193-33) \n	-> the breakout is intended for use with 3.3V and 5V (not needed here)"
 		(exclude_from_sim no)
 		(at 12.7 12.7 0)
-		(size 127 30.48)
+		(size 127 35.56)
 		(margins 0.9525 0.9525 0.9525 0.9525)
 		(stroke
@@
 			)
 			(justify left top)
-			(href "https://files.waveshare.com/upload/8/8e/E-Paper_Driver_HAT.pdf")
 		)
 	)

Commit message: Bigger Zener, improved BoM, general improvements
Parts:
- C10, C11, C13, C6, C7, C8, C9: DigiKey (none) -> 1276-3091-1-ND; Manufacturer PartNo (none) -> CL31B105KBHNFNE
- C12: DigiKey (none) -> 1276-1804-1-ND; Manufacturer PartNo (none) -> CL31B106KAHNNNE
- C4, C5: DigiKey (none) -> 1276-3179-1-ND; Manufacturer PartNo (none) -> CL31B475KBHNFNE
- D7, D8, D9: DigiKey (none) -> MBR0530T1GOSCT-ND; Manufacturer PartNo (none) -> MBR0530T1G
- J6: DigiKey (none) -> 2073-FFC2B28-24-GCT-ND; Manufacturer PartNo (none) -> FFC2B28-24-G
- L1: DigiKey (none) -> 541-1406-1-ND; Manufacturer PartNo (none) -> IFSC1515AHER100M01
- Q4: DigiKey (none) -> BSS138LT3GOSCT-ND; Manufacturer PartNo (none) -> BSS138LT3G
- R10: DigiKey (none) -> 311-10.0KFRCT-ND; Manufacturer PartNo (none) -> RC1206FR-0710KL
- R11: DigiKey (none) -> 273-KDV12DR470ETCT-ND; Manufacturer PartNo (none) -> KDV12DR470ET
