File: ZEReader-Pico.kicad_sch (KiCad schematic)
At the start: 4 parts

Commit message: Reworked v2 routing
- some general improvements
- reworked component numbering
- routed and tuned differential pair (USB)
- added stiching vias and improved ground fills
Parts:
- removed H1, H2, H3, H4: MountingHole, MountingHole:MountingHole_3.2mm_M3_Pad_Via, symbol Mechanical:MountingHole
- added H1, H2, H3, H4: MountingHole_Pad, MountingHole:MountingHole_3.2mm_M3_Pad_Via, symbol Mechanical:MountingHole_Pad
Connections:
- new net GND: H1.1, H2.1, H3.1, H4.1

Commit message: Reworked the PCB after review
Other:
- sheet 01_MCU ports: added none; removed SD_DET_A
- sheet 04_SD-Card ports: added none; removed SD_DET_A
Changed lines of the file:
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@@
+	(wire
+		(pts
+			(xy 76.2 90.17) (xy 101.6 90.17)
+		)
+		(stroke
+			(width 0)
+			(type default)
+		)
+	)
 	(wire
 		(pts
 			(xy 152.4 97.79) (xy 177.8 97.79)
-		)
-		(stroke
-			(width 0)
-			(type default)
-		)
-	)
-	(wire
-		(pts
-			(xy 76.2 90.17) (xy 101.6 90.17)
-		)
-		(stroke
-			(width 0)
-			(type default)
-		)
-	)
-	(wire
-		(pts
-			(xy 152.4 100.33) (xy 177.8 100.33)
 		)
 		(stroke
@@
 			)
 		)
-		(pin "SD_DET_A" bidirectional
+		(pin "SD_DET_B" bidirectional
 			(at 177.8 97.79 180)
-			(effects
-				(font
-					(size 1.27 1.27)
-				)
-				(justify left)
-			)
-		)
-		(pin "SD_DET_B" bidirectional
-			(at 177.8 100.33 180)
 			(effects
 				(font
@@
 			)
 		)
-		(pin "SD_DET_A" bidirectional
+		(pin "SD_DET_B" bidirectional
 			(at 152.4 97.79 0)
 			(effects
 				(font
-					(size 1.27 1.27)
-				)
-				(justify right)
-			)
-		)
-		(pin "SD_DET_B" bidirectional
-			(at 152.4 100.33 0)
-			(effects
-				(font

Commit message: Add proper charging detection, fix zener footprint
Connect the BQ25 status pin to the microcontroller for a proper
charging detection (low active).
Correct the footprint for the selected zener diode.
Somehow, the wrong footprint got assigned.
Other:
- sheet 01_MCU ports: added CHARGING; removed none
- sheet 02a_USB-Battery-Charging ports: added CHARGING; removed none
Changed lines of the file:
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@@
+	(wire
+		(pts
+			(xy 76.2 59.69) (xy 101.6 59.69)
+		)
+		(stroke
+			(width 0)
+			(type default)
+		)
+	)
 	(wire
 		(pts
@@
 			)
 		)
+		(pin "CHARGING" input
+			(at 101.6 59.69 180)
+			(effects
+				(font
+					(size 1.27 1.27)
+				)
+				(justify left)
+			)
+		)
 		(instances
 			(project "ZEReader-Pico"
@@
 			)
 		)
+		(pin "CHARGING" output
+			(at 76.2 59.69 0)
+			(effects
+				(font
+					(size 1.27 1.27)
+				)
+				(justify right)
+			)
+		)

Commit message: Add an voltage bypass mode when USB-C is connected
When USB-C is connected, the device should be charging, but also powered,
without taking care of the on/off button's state.
Otherwise, flashing the device via USB-C would only be
possible as long as the button is pressed which makes the usage
experience a mess and flaky.
This uses p-MOSFETs to do the switch and
a) avoid a battery voltage going to the system when USB-C is connected
b) avoid powering having both, USB-C and Micro-USB active

TODO: This adds the basic idea, routing must be fixed!
Other:
- sheet 02a_USB-Battery-Charging ports: added USB_VBUS; removed none
- sheet 02b_Power-On-Off ports: added USB_VBUS; removed none
Changed lines of the file:
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@@
+	(wire
+		(pts
+			(xy 45.72 60.96) (xy 45.72 81.28)
+		)
+		(stroke
+			(width 0)
+			(type default)
+		)
+	)
+	(wire
+		(pts
+			(xy 76.2 85.09) (xy 101.6 85.09)
+		)
+		(stroke
+			(width 0)
+			(type default)
+		)
+	)
 	(wire
 		(pts
@@
 	(wire
 		(pts
+			(xy 45.72 81.28) (xy 50.8 81.28)
+		)
+		(stroke
+			(width 0)
+			(type default)
+		)
+	)
+	(wire
+		(pts
 			(xy 152.4 119.38) (xy 177.8 119.38)
 		)
@@
 	(wire
 		(pts
-			(xy 76.2 85.09) (xy 101.6 85.09)
-		)
-		(stroke
-			(width 0)
-			(type default)
-		)
-	)
-	(wire
-		(pts
 			(xy 152.4 116.84) (xy 177.8 116.84)
 		)
@@
 		(pts
 			(xy 152.4 57.15) (xy 177.8 57.15)
+		)
+		(stroke
+			(width 0)
+			(type default)
+		)
+	)
+	(wire
+		(pts
+			(xy 50.8 60.96) (xy 45.72 60.96)
 		)
 		(stroke
@@
 			)
 		)
+		(pin "USB_VBUS" output
+			(at 50.8 60.96 180)
+			(effects
+				(font
+					(size 1.27 1.27)
+				)
+				(justify left)
+			)
+		)
 		(instances
 			(project "ZEReader-Pico"
@@
 			)
 		)
+		(pin "USB_VBUS" input
+			(at 50.8 81.28 180)
+			(effects
+				(font
+					(size 1.27 1.27)
+				)
+				(justify left)
+			)
+		)
